File: nerve_gps_pcb.kicad_sch (KiCad schematic)
At the start: 20 parts, among them J1 BF080-16-A-1-L-C, J2 WS2812B, J3 5V GPIO Breakout, U1 SAM-M10Q, U2 TXB0104QPWRQ1

Commit message: Fix #2
Connections:
- net GPS_UART_RX: now also U1.14 (RXD); no longer U1.13 (TXD)
- net GPS_UART_TX: now also U1.13 (TXD); no longer U1.14 (RXD)
Changed lines of the file:
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@@
+		)
+	)
+	(hierarchical_label "GPS_UART_RX"
+		(shape input)
+		(at 85.09 48.26 180)
+		(effects
+			(font
+				(size 1.27 1.27)
+			)
+			(justify right)
+		)
+	)
+	(hierarchical_label "GPS_UART_TX"
+		(shape input)
+		(at 123.19 48.26 0)
+		(effects
+			(font
+				(size 1.27 1.27)
+			)
+			(justify left)
 		)
 	)
@@
 		(shape input)
 		(at 196.85 142.24 180)
-		(fields_autoplaced yes)
 		(effects
 			(font
@@
 		(shape input)
 		(at 50.8 34.29 0)
-		(fields_autoplaced yes)
 		(effects
 			(font
@@
 		(shape input)
 		(at 38.1 34.29 180)
-		(fields_autoplaced yes)
 		(effects
 			(font
@@
 		(shape input)
 		(at 196.85 137.16 180)
-		(fields_autoplaced yes)
 		(effects
 			(font
@@
 		(shape input)
 		(at 85.09 30.48 180)
-		(fields_autoplaced yes)
 		(effects
 			(font
@@
 		(shape input)
 		(at 38.1 31.75 180)
-		(fields_autoplaced yes)
 		(effects
 			(font
@@
 		(shape input)
 		(at 50.8 36.83 0)
-		(fields_autoplaced yes)
 		(effects
 			(font
@@
 		(shape input)
 		(at 86.36 87.63 180)
-		(fields_autoplaced yes)
 		(effects
 			(font
@@
 		(shape input)
 		(at 38.1 39.37 180)
-		(fields_autoplaced yes)
 		(effects
 			(font
@@
 		(shape input)
 		(at 29.21 90.17 180)
-		(fields_autoplaced yes)
 		(effects
 			(font
@@
 		)
 	)
-	(hierarchical_label "GPS_UART_RX"
-		(shape input)
-		(at 123.19 48.26 0)
-		(fields_autoplaced yes)
-		(effects
-			(font
-				(size 1.27 1.27)
-			)
-			(justify left)
-		)
-	)
 	(hierarchical_label "GPIO_1"
 		(shape input)
 		(at 50.8 31.75 0)
-		(fields_autoplaced yes)
 		(effects
 			(font
@@
 		(shape input)
 		(at 29.21 87.63 180)
-		(fields_autoplaced yes)
-		(effects
-			(font
-				(size 1.27 1.27)
-			)
-			(justify right)
-		)
-	)
-	(hierarchical_label "GPS_UART_TX"
-		(shape input)
-		(at 85.09 48.26 180)
-		(fields_autoplaced yes)
 		(effects
 			(font
@@
 		(shape input)
 		(at 196.85 139.7 180)
-		(fields_autoplaced yes)
 		(effects
 			(font
@@
 		(shape input)
 		(at 52.07 90.17 0)
-		(fields_autoplaced yes)
 		(effects
 			(font
@@
 		(shape input)
 		(at 50.8 41.91 0)
-		(fields_autoplaced yes)
 		(effects
 			(font
@@
 		(shape input)
 		(at 29.21 92.71 180)
-		(fields_autoplaced yes)
 		(effects
 			(font
@@
 		(shape input)
 		(at 52.07 92.71 0)
-		(fields_autoplaced yes)
 		(effects
 			(font
@@
 		(shape input)
 		(at 52.07 87.63 0)
-		(fields_autoplaced yes)
 		(effects
 			(font
